Commit message: Complex movement works

File: ROS/arm_control/urdf/env.urdf (robot description, URDF)
Before this commit: robot cells_env, 103 links, 102 joints
Joints:
- joint table_0_joint: origin xyz=-2.0 0.0 0.0 rpy=1.57 0.0 0.0 -> xyz=-2.0 -0.5 0.0 rpy=1.57 0.0 0.0

File: ROS/arm_control/urdf/env.urdf.xacro (robot description, xacro)
@@ -20,5 +20,5 @@
 	</joint>
   <xacro:add_table id="0" parent="foodcort" scale="${mesh_scale_val}">
-    <origin rpy="1.57 0.0 0.0" xyz="-2.0 0.0 0.0" />
+    <origin rpy="1.57 0.0 0.0" xyz="-2.0 -0.5 0.0" />
   </xacro:add_table>
   <xacro:cells_group_macro id="0" parent="foodcort" x_size="4" z_size="3" scale="${mesh_scale_val}">
